File: KiCAD Files/TFG.kicad_pcb (KiCad board)
At the start: 2 copper layers, 70 x 64.5 mm, 47 parts, among them J1 Screw_Terminal_01x03, J2 Screw_Terminal_01x03, J3 Screw_Terminal_01x03, J4 Screw_Terminal_01x02, J5 Screw_Terminal_01x02, Q1 2N3906, Q2 2N3906, Q3 2N3906, Q4 2N3904, Q5 2N3904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

Commit message: add
Parts:
- moved REF2342344 0.25 mm to (165.2, 55.5)
Other:
- outline, holes or cut-outs redrawn
Changed lines of the file:
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@@
   )
   (footprint "MountingHole:MountingHole_2.5mm" (layer "F.Cu")
-    (at 165 55.5)
+    (at 165.25 55.5)
     (descr "Mounting Hole 2.5mm, no annular")
     (tags "mounting hole 2.5mm no annular")
@@
     )
   )
-  (gr_rect (start 98.25 52.555) (end 168.25 117.055) (layer "Edge.Cuts") (width 0.25) (fill none))
+  (gr_line (start 165.25 52.5) (end 98.25 52.55) (layer "Edge.Cuts") (width 0.15))
+  (gr_arc (start 168.25 114.02868) (mid 167.35755 116.151284) (end 165.22868 117.02868) (layer "Edge.Cuts") (width 0.15))
+  (gr_line (start 98.25 117.05) (end 165.22868 117.02868) (layer "Edge.Cuts") (width 0.15))
+  (gr_arc (start 165.25 52.5) (mid 167.37132 53.37868) (end 168.25 55.5) (layer "Edge.Cuts") (width 0.15))
+  (gr_line (start 168.25 114.02868) (end 168.25 55.5) (layer "Edge.Cuts") (width 0.15))
+  (gr_line (start 98.25 52.55) (end 98.25 117.05) (layer "Edge.Cuts") (width 0.15))
   (segment (start 150.24952 75.75) (end 148.2948 75.75) (width 1.3) (layer "F.Cu") (net 1))
   (segment (start 110.8125 78.8) (end 109.95 78.8) (width 1.3) (layer "F.Cu") (net 1))
